Commit message: debug

File: src/ros2_foundry_description/urdf/arm.urdf.xacro (robot description, xacro)
@@ -2,68 +2,43 @@
 <robot xmlns:xacro="http://www.ros.org/wiki/xacro">
   <xacro:macro name="robot_arm" params="prefix parent *origin">
-    <joint name="${prefix}arm_base_joint" type="fixed">
-      <parent link="${parent}"/>
-      <child link="${prefix}arm_base_link"/>
-      <xacro:insert_block name="origin"/>
-    </joint>
+    <joint name="${prefix}arm_base_joint" type="fixed"><parent link="${parent}"/><child link="${prefix}arm_base_link"/><xacro:insert_block name="origin"/></joint>
     <link name="${prefix}arm_base_link">
-      <visual>
-        <geometry>
-          <cylinder radius="0.07" length="0.05"/>
-        </geometry>
-        <material name="grey"/>
-      </visual>
-      <collision>
-        <geometry>
-          <cylinder radius="0.07" length="0.05"/>
-        </geometry>
-      </collision>
+      <visual><geometry><cylinder radius="0.07" length="0.05"/></geometry><material name="grey"/></visual>
+      <collision><geometry><cylinder radius="0.07" length="0.05"/></geometry></collision>
+      <inertial><mass value="0.5"/><inertia ixx="0.01" ixy="0" ixz="0" iyy="0.01" iyz="0" izz="0.01"/></inertial>
     </link>
-    <!-- Arm Joints and Links -->
     <xacro:macro name="arm_joint" params="name parent child joint_type axis_xyz origin_xyz limit_lower limit_upper">
-      <joint name="${name}" type="${joint_type}">
-        <parent link="${parent}"/>
-        <child link="${child}"/>
-        <origin xyz="${origin_xyz}" rpy="0 0 0"/>
-        <axis xyz="${axis_xyz}"/>
-        <limit lower="${limit_lower}" upper="${limit_upper}" effort="100" velocity="1.0"/>
-      </joint>
+      <joint name="${name}" type="${joint_type}"><parent link="${parent}"/><child link="${child}"/><origin xyz="${origin_xyz}" rpy="0 0 0"/><axis xyz="${axis_xyz}"/><limit lower="${limit_lower}" upper="${limit_upper}" effort="100" velocity="1.0"/></joint>
     </xacro:macro>
-    <xacro:macro name="arm_link" params="name length radius">
+    <xacro:macro name="arm_link" params="name length radius mass">
        <link name="${name}">
-        <visual>
-          <geometry>
-            <cylinder radius="${radius}" length="${length}"/>
-          </geometry>
-          <origin xyz="0 0 ${length/2}" rpy="0 0 0"/>
-          <material name="blue"/>
-        </visual>
-        <collision>
-          <geometry>
-            <cylinder radius="${radius}" length="${length}"/>
-          </geometry>
-           <origin xyz="0 0 ${length/2}" rpy="0 0 0"/>
-        </collision>
+        <visual><geometry><cylinder radius="${radius}" length="${length}"/></geometry><origin xyz="0 0 ${length/2}" rpy="0 0 0"/><material name="blue"/></visual>
+        <collision><geometry><cylinder radius="${radius}" length="${length}"/></geometry><origin xyz="0 0 ${length/2}" rpy="0 0 0"/></collision>
+        <inertial><mass value="${mass}"/><inertia ixx="0.01" ixy="0" ixz="0" iyy="0.01" iyz="0" izz="0.01"/></inertial>
       </link>
     </xacro:macro>
-    <!-- Joint 1 -->
     <xacro:arm_joint name="${prefix}joint1" parent="${prefix}arm_base_link" child="${prefix}link1" joint_type="revolute" axis_xyz="0 0 1" origin_xyz="0 0 0.025" limit_lower="-${PI}" limit_upper="${PI}"/>
-    <xacro:arm_link name="${prefix}link1" length="0.2" radius="0.05"/>
-    <!-- Joint 2 -->
+    <xacro:arm_link name="${prefix}link1" length="0.2" radius="0.05" mass="1.0"/>
     <xacro:arm_joint name="${prefix}joint2" parent="${prefix}link1" child="${prefix}link2" joint_type="revolute" axis_xyz="0 1 0" origin_xyz="0 0 0.2" limit_lower="-${PI/2}" limit_upper="${PI/2}"/>
-    <xacro:arm_link name="${prefix}link2" length="0.3" radius="0.05"/>
-    <!-- Joint 3 -->
+    <xacro:arm_link name="${prefix}link2" length="0.3" radius="0.05" mass="1.5"/>
     <xacro:arm_joint name="${prefix}joint3" parent="${prefix}link2" child="${prefix}link3" joint_type="revolute" axis_xyz="0 1 0" origin_xyz="0 0 0.3" limit_lower="-${PI/2}" limit_upper="${PI/2}"/>
-    <xacro:arm_link name="${prefix}link3" length="0.25" radius="0.05"/>
-    <!-- Joint 4 -->
+    <xacro:arm_link name="${prefix}link3" length="0.25" radius="0.05" mass="1.2"/>
     <xacro:arm_joint name="${prefix}joint4" parent="${prefix}link3" child="${prefix}link4" joint_type="revolute" axis_xyz="1 0 0" origin_xyz="0 0 0.25" limit_lower="-${PI}" limit_upper="${PI}"/>
-    <xacro:arm_link name="${prefix}link4" length="0.1" radius="0.05"/>
-    <!-- Joint 5 -->
+    <xacro:arm_link name="${prefix}link4" length="0.1" radius="0.05" mass="0.5"/>
     <xacro:arm_joint name="${prefix}joint5" parent="${prefix}link4" child="${prefix}link5" joint_type="revolute" axis_xyz="0 1 0" origin_xyz="0 0 0.1" limit_lower="-${PI/2}" limit_upper="${PI/2}"/>
-    <xacro:arm_link name="${prefix}link5" length="0.1" radius="0.05"/>
-    <!-- Joint 6 -->
+    <xacro:arm_link name="${prefix}link5" length="0.1" radius="0.05" mass="0.5"/>
     <xacro:arm_joint name="${prefix}joint6" parent="${prefix}link5" child="${prefix}tool0" joint_type="revolute" axis_xyz="1 0 0" origin_xyz="0 0 0.1" limit_lower="-${PI}" limit_upper="${PI}"/>
-    <!-- Tool frame -->
-    <link name="${prefix}tool0"/>
+    <!-- ==================================================== -->
+    <!-- == VITAL FIX: ADDED INERTIAL TAG TO tool0 LINK    == -->
+    <!-- ==================================================== -->
+    <link name="${prefix}tool0">
+      <inertial>
+        <mass value="0.001" />
+        <inertia ixx="0.0001" ixy="0.0" ixz="0.0" iyy="0.0001" iyz="0.0" izz="0.0001" />
+      </inertial>
+    </link>
+    <!-- ==================================================== -->
+    <!-- ============ END OF VITAL FIX ====================== -->
+    <!-- ==================================================== -->
   </xacro:macro>
 </robot>

File: src/ros2_foundry_description/urdf/base.urdf.xacro (robot description, xacro)
@@ -2,5 +2,4 @@
 <robot xmlns:xacro="http://www.ros.org/wiki/xacro">
   <xacro:macro name="mobile_base" params="prefix">
-    <!-- Base Link -->
     <link name="${prefix}base_footprint"/>
     <joint name="${prefix}base_joint" type="fixed">
@@ -10,65 +9,28 @@
     </joint>
     <link name="${prefix}base_link">
-      <visual>
-        <origin xyz="0 0 0" rpy="0 0 0"/>
-        <geometry>
-          <cylinder radius="0.25" length="0.1"/>
-        </geometry>
-        <material name="blue"/>
-      </visual>
-      <collision>
-        <origin xyz="0 0 0" rpy="0 0 0"/>
-        <geometry>
-          <cylinder radius="0.25" length="0.1"/>
-        </geometry>
-      </collision>
+      <visual><geometry><cylinder radius="0.25" length="0.1"/></geometry><material name="blue"/></visual>
+      <collision><geometry><cylinder radius="0.25" length="0.1"/></geometry></collision>
+      <inertial><mass value="5.0"/><inertia ixx="0.1" ixy="0" ixz="0" iyy="0.1" iyz="0" izz="0.1"/></inertial>
     </link>
-    <!-- Wheels -->
-    <xacro:macro name="wheel" params="prefix side y_pos">
-      <joint name="${prefix}${side}_wheel_joint" type="continuous">
-        <parent link="${prefix}base_link"/>
-        <child link="${prefix}${side}_wheel_link"/>
-        <origin xyz="0 ${y_pos} 0" rpy="-${PI/2} 0 0"/>
-        <axis xyz="0 0 1"/>
-      </joint>
+    <xacro:macro name="wheel" params="side y_pos">
+      <joint name="${prefix}${side}_wheel_joint" type="continuous"><parent link="${prefix}base_link"/><child link="${prefix}${side}_wheel_link"/><origin xyz="0 ${y_pos} 0" rpy="-${PI/2} 0 0"/><axis xyz="0 0 1"/></joint>
       <link name="${prefix}${side}_wheel_link">
-        <visual>
-          <geometry>
-            <cylinder radius="0.1" length="0.05"/>
-          </geometry>
-          <material name="black"/>
-        </visual>
-        <collision>
-          <geometry>
-            <cylinder radius="0.1" length="0.05"/>
-          </geometry>
-        </collision>
+        <visual><geometry><cylinder radius="0.1" length="0.05"/></geometry><material name="black"/></visual>
+        <collision><geometry><cylinder radius="0.1" length="0.05"/></geometry></collision>
+        <inertial><mass value="0.5"/><inertia ixx="0.01" ixy="0" ixz="0" iyy="0.01" iyz="0" izz="0.01"/></inertial>
       </link>
     </xacro:macro>
-    <xacro:wheel prefix="${prefix}" side="left" y_pos="0.25"/>
-    <xacro:wheel prefix="${prefix}" side="right" y_pos="-0.25"/>
-    <!-- Caster Wheels -->
-    <xacro:macro name="caster_wheel" params="prefix x_pos">
-        <joint name="${prefix}caster_${x_pos}_joint" type="fixed">
-            <parent link="${prefix}base_link"/>
-            <child link="${prefix}caster_${x_pos}_link"/>
-            <origin xyz="${x_pos} 0 -0.05" rpy="0 0 0"/>
-        </joint>
+    <xacro:wheel side="left" y_pos="0.255"/>
+    <xacro:wheel side="right" y_pos="-0.255"/>
+    <xacro:macro name="caster_wheel" params="x_pos">
+        <joint name="${prefix}caster_${x_pos}_joint" type="fixed"><parent link="${prefix}base_link"/><child link="${prefix}caster_${x_pos}_link"/><origin xyz="${x_pos} 0 -0.05" rpy="0 0 0"/></joint>
         <link name="${prefix}caster_${x_pos}_link">
-            <visual>
-                <geometry>
-                    <sphere radius="0.05"/>
-                </geometry>
-                <material name="black"/>
-            </visual>
-            <collision>
-                <geometry>
-                    <sphere radius="0.05"/>
-                </geometry>
-            </collision>
+            <visual><geometry><sphere radius="0.05"/></geometry><material name="black"/></visual>
+            <collision><geometry><sphere radius="0.05"/></geometry></collision>
+            <inertial><mass value="0.2"/><inertia ixx="0.001" ixy="0" ixz="0" iyy="0.001" iyz="0" izz="0.001"/></inertial>
         </link>
     </xacro:macro>
-    <xacro:caster_wheel prefix="${prefix}" x_pos="0.15"/>
-    <xacro:caster_wheel prefix="${prefix}" x_pos="-0.15"/>
+    <xacro:caster_wheel x_pos="0.15"/>
+    <xacro:caster_wheel x_pos="-0.15"/>
   </xacro:macro>
 </robot>

File: src/ros2_foundry_description/urdf/foundry_bot.urdf.xacro (robot description, xacro)
@@ -1,5 +1,4 @@
 <?xml version="1.0"?>
 <robot name="foundry_bot" xmlns:xacro="http://www.ros.org/wiki/xacro">
-  <!-- Include all parts -->
   <xacro:include filename="$(find ros2_foundry_description)/urdf/common.xacro"/>
   <xacro:include filename="$(find ros2_foundry_description)/urdf/base.urdf.xacro"/>
@@ -7,21 +6,27 @@
   <xacro:include filename="$(find ros2_foundry_description)/urdf/gripper.urdf.xacro"/>
   <xacro:include filename="$(find ros2_foundry_description)/urdf/sensors.urdf.xacro"/>
-  <!-- Instantiate all parts -->
-  <!-- Mobile Base -->
   <xacro:mobile_base prefix=""/>
-  <!-- Arm -->
-  <xacro:robot_arm prefix="" parent="base_link">
-    <origin xyz="0 0 0.05" rpy="0 0 0"/>
-  </xacro:robot_arm>
-  <!-- Gripper -->
-  <xacro:gripper prefix="" parent="tool0">
-    <origin xyz="0 0 0" rpy="0 0 0"/>
-  </xacro:gripper>
-  <!-- Sensors -->
-  <xacro:lidar prefix="" parent="base_link">
-    <origin xyz="0.2 0 0.05" rpy="0 0 0"/>
-  </xacro:lidar>
-  <xacro:depth_camera prefix="" parent="link5">
-    <origin xyz="0 0 0.05" rpy="0 ${PI/2} 0"/>
-  </xacro:depth_camera>
+  <xacro:robot_arm prefix="" parent="base_link"><origin xyz="0 0 0.05" rpy="0 0 0"/></xacro:robot_arm>
+  <xacro:gripper prefix="" parent="tool0"><origin xyz="0 0 0" rpy="0 0 0"/></xacro:gripper>
+  <xacro:lidar prefix="" parent="base_link"><origin xyz="0.2 0 0.05" rpy="0 0 0"/></xacro:lidar>
+  <xacro:depth_camera prefix="" parent="link5"><origin xyz="0 0 0.05" rpy="0 ${PI/2} 0"/></xacro:depth_camera>
+  <ros2_control name="FoundryBotSystem" type="system">
+    <hardware><plugin>gazebo_ros2_control/GazeboSystem</plugin></hardware>
+    <joint name="left_wheel_joint"><command_interface name="velocity"/><state_interface name="position"/><state_interface name="velocity"/></joint>
+    <joint name="right_wheel_joint"><command_interface name="velocity"/><state_interface name="position"/><state_interface name="velocity"/></joint>
+    <joint name="joint1"><command_interface name="position"/><state_interface name="position"/><state_interface name="velocity"/></joint>
+    <joint name="joint2"><command_interface name="position"/><state_interface name="position"/><state_interface name="velocity"/></joint>
+    <joint name="joint3"><command_interface name="position"/><state_interface name="position"/><state_interface name="velocity"/></joint>
+    <joint name="joint4"><command_interface name="position"/><state_interface name="position"/><state_interface name="velocity"/></joint>
+    <joint name="joint5"><command_interface name="position"/><state_interface name="position"/><state_interface name="velocity"/></joint>
+    <joint name="joint6"><command_interface name="position"/><state_interface name="position"/><state_interface name="velocity"/></joint>
+    <joint name="finger_left_joint"><command_interface name="position"/><state_interface name="position"/><state_interface name="velocity"/></joint>
+    <joint name="finger_right_joint"><command_interface name="position"/><state_interface name="position"/><state_interface name="velocity"/></joint>
+  </ros2_control>
+  <gazebo>
+    <plugin filename="libgazebo_ros2_control.so" name="gazebo_ros2_control">
+        <robot_sim_type>gazebo_ros2_control/DefaultRobotHWSim</robot_sim_type>
+        <parameters>$(find ros2_foundry_description)/config/ros2_controllers.yaml</parameters>
+    </plugin>
+  </gazebo>
 </robot>

File: src/ros2_foundry_description/urdf/gripper.urdf.xacro (robot description, xacro)
@@ -2,45 +2,16 @@
 <robot xmlns:xacro="http://www.ros.org/wiki/xacro">
   <xacro:macro name="gripper" params="prefix parent *origin">
-    <joint name="${prefix}gripper_base_joint" type="fixed">
-      <parent link="${parent}"/>
-      <child link="${prefix}gripper_base"/>
-      <xacro:insert_block name="origin"/>
-    </joint>
+    <joint name="${prefix}gripper_base_joint" type="fixed"><parent link="${parent}"/><child link="${prefix}gripper_base"/><xacro:insert_block name="origin"/></joint>
     <link name="${prefix}gripper_base">
-        <visual>
-            <geometry>
-                <box size="0.05 0.1 0.05"/>
-            </geometry>
-            <material name="grey"/>
-        </visual>
-        <collision>
-            <geometry>
-                <box size="0.05 0.1 0.05"/>
-            </geometry>
-        </collision>
+        <visual><geometry><box size="0.05 0.1 0.05"/></geometry><material name="grey"/></visual>
+        <collision><geometry><box size="0.05 0.1 0.05"/></geometry></collision>
+        <inertial><mass value="0.2"/><inertia ixx="0.001" ixy="0" ixz="0" iyy="0.001" iyz="0" izz="0.001"/></inertial>
     </link>
-    <!-- Gripper Fingers -->
     <xacro:macro name="finger" params="side y_pos">
-        <joint name="${prefix}finger_${side}_joint" type="prismatic">
-            <parent link="${prefix}gripper_base"/>
-            <child link="${prefix}finger_${side}_link"/>
-            <origin xyz="0 ${y_pos} 0" rpy="0 0 0"/>
-            <axis xyz="0 1 0"/>
-            <limit lower="0.0" upper="0.04" effort="10" velocity="0.1"/>
-        </joint>
+        <joint name="${prefix}finger_${side}_joint" type="prismatic"><parent link="${prefix}gripper_base"/><child link="${prefix}finger_${side}_link"/><origin xyz="0 ${y_pos} 0" rpy="0 0 0"/><axis xyz="0 1 0"/><limit lower="0.0" upper="0.04" effort="10" velocity="0.1"/></joint>
         <link name="${prefix}finger_${side}_link">
-            <visual>
-                <geometry>
-                    <box size="0.08 0.01 0.02"/>
-                </geometry>
-                <origin xyz="0.04 0 0"/>
-                <material name="black"/>
-            </visual>
-            <collision>
-                <geometry>
-                    <box size="0.08 0.01 0.02"/>
-                </geometry>
-                 <origin xyz="0.04 0 0"/>
-            </collision>
+            <visual><geometry><box size="0.08 0.01 0.02"/></geometry><origin xyz="0.04 0 0"/><material name="black"/></visual>
+            <collision><geometry><box size="0.08 0.01 0.02"/></geometry><origin xyz="0.04 0 0"/></collision>
+            <inertial><mass value="0.05"/><inertia ixx="0.0001" ixy="0" ixz="0" iyy="0.0001" iyz="0" izz="0.0001"/></inertial>
         </link>
     </xacro:macro>

File: src/ros2_foundry_description/urdf/sensors.urdf.xacro (robot description, xacro)
@@ -1,34 +1,18 @@
 <?xml version="1.0"?>
 <robot xmlns:xacro="http://www.ros.org/wiki/xacro">
-  <!-- 2D Lidar -->
   <xacro:macro name="lidar" params="prefix parent *origin">
-    <joint name="${prefix}lidar_joint" type="fixed">
-      <parent link="${parent}"/>
-      <child link="${prefix}lidar_link"/>
-      <xacro:insert_block name="origin"/>
-    </joint>
+    <joint name="${prefix}lidar_joint" type="fixed"><parent link="${parent}"/><child link="${prefix}lidar_link"/><xacro:insert_block name="origin"/></joint>
     <link name="${prefix}lidar_link">
-      <visual>
-        <geometry>
-          <cylinder radius="0.05" length="0.04"/>
-        </geometry>
-        <material name="black"/>
-      </visual>
+      <visual><geometry><cylinder radius="0.05" length="0.04"/></geometry><material name="black"/></visual>
+      <collision><geometry><cylinder radius="0.05" length="0.04"/></geometry></collision>
+      <inertial><mass value="0.1"/><inertia ixx="0.001" ixy="0" ixz="0" iyy="0.001" iyz="0" izz="0.001"/></inertial>
     </link>
   </xacro:macro>
-  <!-- 3D Depth Camera -->
   <xacro:macro name="depth_camera" params="prefix parent *origin">
-    <joint name="${prefix}camera_joint" type="fixed">
-      <parent link="${parent}"/>
-      <child link="${prefix}camera_link"/>
-      <xacro:insert_block name="origin"/>
-    </joint>
+    <joint name="${prefix}camera_joint" type="fixed"><parent link="${parent}"/><child link="${prefix}camera_link"/><xacro:insert_block name="origin"/></joint>
     <link name="${prefix}camera_link">
-      <visual>
-        <geometry>
-          <box size="0.02 0.08 0.03"/>
-        </geometry>
-        <material name="black"/>
-      </visual>
+      <visual><geometry><box size="0.02 0.08 0.03"/></geometry><material name="black"/></visual>
+      <collision><geometry><box size="0.02 0.08 0.03"/></geometry></collision>
+      <inertial><mass value="0.05"/><inertia ixx="0.0001" ixy="0" ixz="0" iyy="0.0001" iyz="0" izz="0.0001"/></inertial>
     </link>
   </xacro:macro>
